File: MINI_SAM_D51_007.brd (EAGLE design)
At the start: 24.1 x 40.4 mm, 32 parts, among them IC2 PRTR5V0U2X, IC4 ATSAMD51G_TQFN48, J1 MOLEX_47346-100147346, J2 CORTEX_DEBUG_PTH, SW1 KMS233GLFG, SW2 KMS233GLFG, U1 GD25x16

Commit message: Slight Update to Rev 007
Other:
- board size 24.1 x 40.4 mm -> 25.4 x 40.4 mm

Commit message: Name Changes
Parts:
- removed IC4: ATSAMD51G_TQFN48, microbuilder:TQFN48_7MM
- added U2: GD25x16, microbuilder:USON8
- U1: value GD25x16 -> ATSAMD51G_TQFN48; device microbuilder:USON8 -> microbuilder:TQFN48_7MM
- moved U1 5.91 mm to (12.0, 20.0), turned to 45 degrees
- renumbered IC2 to IC1
Connections:
- net !RESET: now also U1.40; no longer IC4.40
- net A0: now also U1.3; no longer IC4.3
- net A1: now also U1.10; no longer IC4.10
- net A2: now also U1.7; no longer IC4.7
- net A3: now also U1.8; no longer IC4.8
- net A4: now also U1.9; no longer IC4.9
- net A5: now also U1.11; no longer IC4.11
- net A6_D2: now also U1.12; no longer IC4.12
- net AREF: now also U1.4; no longer IC4.4
- net D10: now also U1.29; no longer IC4.29
- net D11: now also U1.30; no longer IC4.30
- net D12: now also U1.32; no longer IC4.32
- net D13: now also U1.31; no longer IC4.31
- net D3: now also U1.37; no longer IC4.37
- net D4: now also U1.23; no longer IC4.23
- net D5: now also U1.24; no longer IC4.24
- net D9: now also U1.28; no longer IC4.28
- net DOTSTAR_CLK: now also U1.47; no longer IC4.47
- net DOTSTAR_DATA: now also U1.48; no longer IC4.48
- net GND: now also U1.18, U1.35, U1.42, U1.5, U1.THERMAL, U2.4; no longer IC4.18, IC4.35, IC4.42, IC4.5, IC4.THERMAL, U1.4
- net MISO: now also U1.38; no longer IC4.38
- net MOSI: now also U1.1; no longer IC4.1
- net N$9: now also U1.41; no longer IC4.41
- net QSPI_CS: now also U1.20, U2.1; no longer IC4.20, U1.1
- net QSPI_DATA[0]: now also U1.13, U2.5; no longer IC4.13, U1.5
- net QSPI_DATA[1]: now also U1.14, U2.2; no longer IC4.14, U1.2
- net QSPI_DATA[2]: now also U1.15, U2.3; no longer IC4.15, U1.3
- net QSPI_DATA[3]: now also U1.16, U2.7; no longer IC4.16, U1.7
- net QSPI_SCK: now also U1.19, U2.6; no longer IC4.19, U1.6
- net RX_D0: now also U1.25; no longer IC4.25
- net SCK: now also U1.2; no longer IC4.2
- net SCL: now also U1.22; no longer IC4.22
- net SDA: now also U1.21; no longer IC4.21
- net SWCLK: now also U1.45; no longer IC4.45
- net SWDIO: now also U1.46; no longer IC4.46
- net TX_D1: now also U1.26; no longer IC4.26
- net USBD+: now also U1.34; no longer IC4.34
- net USBD-: now also U1.33; no longer IC4.33
- net VDD: now also U1.17, U1.36, U1.44, U2.8; no longer IC4.17, IC4.36, IC4.44, U1.8
- net VDDANA: now also U1.6; no longer IC4.6
- net VSW: now also U1.43; no longer IC4.43
