File: MINI_SAM_D51_007.sch (EAGLE design)
At the start: 31 parts, among them IC2 PRTR5V0U2X, IC4 ATSAMD51G_TQFN48, J1 MOLEX_47346-100147346, J2 CORTEX_DEBUG_PTH, SW1 KMS233GLFG, SW2 KMS233GLFG, U1 GD25x16

Commit message: Name Changes
Parts:
- removed IC4: ATSAMD51G_TQFN48, microbuilder:ATSAMD51G_TQFN48
- added U2: GD25x16, microbuilder:SPIFLASH_8PINUX
- U1: value GD25x16 -> ATSAMD51G_TQFN48; device microbuilder:SPIFLASH_8PINUX -> microbuilder:ATSAMD51G_TQFN48
- renumbered IC2 to IC1
Connections:
- net !RESET: now also U1G$1./RESET; no longer IC4G$1./RESET
- net A0: now also U1G$1.PA02/EINT2/AIN0/VOUT0; no longer IC4G$1.PA02/EINT2/AIN0/VOUT0
- net A1: now also U1G$1.PA05/I5/AIN5/VOUT1/SERCOM0.1; no longer IC4G$1.PA05/I5/AIN5/VOUT1/SERCOM0.1
- net A2: now also U1G$1.PB08/I8/AIN2/SERCOM4.0; no longer IC4G$1.PB08/I8/AIN2/SERCOM4.0
- net A3: now also U1G$1.PB09/I9/AIN3/SERCOM4.1; no longer IC4G$1.PB09/I9/AIN3/SERCOM4.1
- net A4: now also U1G$1.PA04/I4/VREFB/AIN4/SERCOM0.0; no longer IC4G$1.PA04/I4/VREFB/AIN4/SERCOM0.0
- net A5: now also U1G$1.PA06/I6/VREFC/AIN6/SERCOM0.2; no longer IC4G$1.PA06/I6/VREFC/AIN6/SERCOM0.2
- net A6_D2: now also U1G$1.PA07/I7/AIN7/SERCOM0.3; no longer IC4G$1.PA07/I7/AIN7/SERCOM0.3
- net AREF: now also U1G$1.PA03/I3/VREFA/AIN1; no longer IC4G$1.PA03/I3/VREFA/AIN1
- net D10: now also U1G$1.PA20/I4/SERCOM3+5.2/I2SFS0; no longer IC4G$1.PA20/I4/SERCOM3+5.2/I2SFS0
- net D11: now also U1G$1.PA21/I5/SERCOM3+5.3/I2SDO; no longer IC4G$1.PA21/I5/SERCOM3+5.3/I2SDO
- net D12: now also U1G$1.PA23/I2C/I7/SERCOM3.1+5.0/SOF/I2SFS1; no longer IC4G$1.PA23/I2C/I7/SERCOM3.1+5.0/SOF/I2SFS1
- net D13: now also U1G$1.PA22/I2C/I6/SERCOM3.0+5.1/I2SDI; no longer IC4G$1.PA22/I2C/I6/SERCOM3.0+5.1/I2SDI
- net D3: now also U1G$1.PB22/I6/SERCOM1+5.2; no longer IC4G$1.PB22/I6/SERCOM1+5.2
- net D4: now also U1G$1.PA14/I14/SERCOM2+4.2; no longer IC4G$1.PA14/I14/SERCOM2+4.2
- net D5: now also U1G$1.PA15/I15/SERCOM2+4.3; no longer IC4G$1.PA15/I15/SERCOM2+4.3
- net D9: now also U1G$1.PA19/I3/SERCOM1+3.3; no longer IC4G$1.PA19/I3/SERCOM1+3.3
- net DOTSTAR_CLK: now also U1G$1.PB02/I2/AIN14/SERCOM5.0; no longer IC4G$1.PB02/I2/AIN14/SERCOM5.0
- net DOTSTAR_DATA: now also U1G$1.PB03/I3/AIN15/SERCOM5.1; no longer IC4G$1.PB03/I3/AIN15/SERCOM5.1
- net GND: now also U1G$1.GND, U1G$1.GNDA, U1G$3.TP, U2.VSS; no longer IC4G$1.GND, IC4G$1.GNDA, IC4G$3.TP, U1.VSS
- net MISO: now also U1G$1.PB23/I7/SERCOM1+5.3; no longer IC4G$1.PB23/I7/SERCOM1+5.3
- net MOSI: now also U1G$1.PA00/EINT0/SERCOM1.0; no longer IC4G$1.PA00/EINT0/SERCOM1.0
- net N$9: now also U1G$1.VDDCORE; no longer IC4G$1.VDDCORE
- net QSPI_CS: now also U1G$1.PB11/I11/SERCOM4.3/I2SFS1, U2.SSEL; no longer IC4G$1.PB11/I11/SERCOM4.3/I2SFS1, U1.SSEL
- net QSPI_DATA[0]: now also U1G$1.PA08/I2C/AIN8/SERCOM0.0+2.1/I2SMCK, U2.MOSI; no longer IC4G$1.PA08/I2C/AIN8/SERCOM0.0+2.1/I2SMCK, U1.MOSI
- net QSPI_DATA[1]: now also U1G$1.PA09/I2C/I9/AIN9/SERCOM0.1+2.0/I2SFS0, U2.MISO; no longer IC4G$1.PA09/I2C/I9/AIN9/SERCOM0.1+2.0/I2SFS0, U1.MISO
- net QSPI_DATA[2]: now also U1G$1.PA10/I10/AIN10/SERCOM0+2.2/I2SCK, U2.WP#/IO2; no longer IC4G$1.PA10/I10/AIN10/SERCOM0+2.2/I2SCK, U1.WP#/IO2
- net QSPI_DATA[3]: now also U1G$1.PA11/I11/AIN11/SERCOM0+2.3/I2SDO, U2.HOLD#/IO3; no longer IC4G$1.PA11/I11/AIN11/SERCOM0+2.3/I2SDO, U1.HOLD#/IO3
- net QSPI_SCK: now also U1G$1.PB10/I10/SERCOM4.2/I2SDI, U2.SCK; no longer IC4G$1.PB10/I10/SERCOM4.2/I2SDI, U1.SCK
- net RX_D0: now also U1G$1.PA16/I2C/I0/SERCOM1.0+3.1; no longer IC4G$1.PA16/I2C/I0/SERCOM1.0+3.1
- net SCK: now also U1G$1.PA01/EINT1/SERCOM1.1; no longer IC4G$1.PA01/EINT1/SERCOM1.1
- net SCL: now also U1G$1.PA13/I13/I2C/SERCOM2.1+4.0; no longer IC4G$1.PA13/I13/I2C/SERCOM2.1+4.0
- net SDA: now also U1G$1.PA12/I12/I2C/SERCOM2.0+4.1; no longer IC4G$1.PA12/I12/I2C/SERCOM2.0+4.1
- net SWCLK: now also U1G$1.PA30/I14/SECOM1.2/SWCLK; no longer IC4G$1.PA30/I14/SECOM1.2/SWCLK
- net SWDIO: now also U1G$1.PA31/I15/SECOM1.3/SWDIO; no longer IC4G$1.PA31/I15/SECOM1.3/SWDIO
- net TX_D1: now also U1G$1.PA17/I2C/I1/SERCOM1.1+3.0; no longer IC4G$1.PA17/I2C/I1/SERCOM1.1+3.0
- net USBD+: now also U1G$1.PA25/I9/SERCOM3+5.3/D+; no longer IC4G$1.PA25/I9/SERCOM3+5.3/D+
- net USBD-: now also U1G$1.PA24/I8/SERCOM3+5.2/D-; no longer IC4G$1.PA24/I8/SERCOM3+5.2/D-
- net VDD: now also U1G$1.VDDIO, U2.VCC; no longer IC4G$1.VDDIO, U1.VCC
- net VDDANA: now also U1G$1.VDDA; no longer IC4G$1.VDDA
