File: MINI_SAM_D51_009.brd (EAGLE design)
At the start: 25.4 x 40.4 mm, 32 parts, among them IC2 PRTR5V0U2X, IC4 ATSAMD51G_TQFN48, J1 MOLEX_47346-100147346, J2 CORTEX_DEBUG_PTH, SW1 KMS233GLFG, SW2 KMS233GLFG, U1 GD25x16

Commit message: Adding revisions
Parts:
- added J5: 1X8_HEADER_1.27MM, Shockley_Custom:1X8_HEADER_1.27MM
- J2: value CORTEX_DEBUG_PTH -> 1X5_HEADER_1.27MM; device SparkFun-Connectors:2X5-PTH-1.27MM -> Shockley_Custom:1X5_HEADER_1.27MM
- J3: value (none) -> 1X8_HEADER_1.27MM; device pinhead+:1X11_SMT -> Shockley_Custom:1X8_HEADER_1.27MM
- J4: value (none) -> 1X5_HEADER_1.27MM; device pinhead+:1X11_SMT -> Shockley_Custom:1X5_HEADER_1.27MM
- moved J4 15.1 mm to (22.3, 19.2), flipped to the top, turned to 281.5 degrees
- moved J3 11.6 mm to (5.60, 8.25), flipped to the top, turned to 267.8 degrees
- moved J2 1.89 mm to (1.70, 19.2), turned to 258.5 degrees
- moved C11 0.93 mm to (20.7, 16.4)
- moved VREG 0.60 mm to (20.1, 19.6)
- moved SW1 0.15 mm to (8.07, 1.65)
- moved SW2 0.15 mm to (15.9, 1.65)
Connections:
- removed net A6_D2: IC4.12, J3.8
- removed net D10: IC4.29
- removed net D11: IC4.30
- removed net D9: IC4.28, R5.2, SW2.3, SW2.4
- new net A6: IC4.12, J5.P$1
- new net BUTTON_D6: IC4.1, R5.2, SW2.2, SW2.3
- net !RESET: now also J2.P$3; no longer J2.10, J4.8
- net A0: now also J5.P$7; no longer J3.2
- net A1: now also IC4.7, J5.P$6; no longer IC4.10, J3.3
- net A2: now also IC4.8, J5.P$5; no longer IC4.7, J3.4
- net A3: now also IC4.9, J5.P$4; no longer IC4.8, J3.5
- net A4: now also IC4.10, J5.P$3; no longer IC4.9, J3.6
- net A5: now also J5.P$2; no longer J3.7
- net AREF: now also J5.P$8; no longer J3.1
- net D3: now also IC4.28, J3.P$3; no longer IC4.37, J4.5
- net D4: now also IC4.29, J3.P$4; no longer IC4.23, J4.4
- net D5: now also IC4.30, J3.P$5; no longer IC4.24, J4.3
- net GND: now also J2.P$5, J4.P$5; no longer J2.3, J2.5, J3.11
- net MISO: now also J3.P$7; no longer J4.10
- net MOSI: now also IC4.37, J3.P$6; no longer IC4.1, J4.9
- net RX_D0: now also J3.P$1; no longer J4.1
- net SCK: now also J3.P$8; no longer J4.11
- net SCL: now also J4.P$1; no longer J4.6
- net SDA: now also J4.P$2; no longer J4.7
- net SWCLK: now also J2.P$2; no longer J2.4
- net SWDIO: now also J2.P$1; no longer J2.2
- net TX_D1: now also J3.P$2; no longer J4.2
- net VDD: now also J2.P$4, J4.P$4, SW2.1; no longer J2.1, J3.9, SW2.5
- net VIN: now also J4.P$3; no longer J3.10
Routing:
- net D9: track 40.6 -> 0.00 mm, vias 4 -> 0
- net TX_D1: track 1.79 -> 22.5 mm, vias 1 -> 2
- net VDD: track 86.6 -> 66.1 mm, vias 7 -> 6
- net BUTTON_D6: track 0.00 -> 16.0 mm, vias 0 -> 2
- net D3: track 3.71 -> 19.7 mm
- net AREF: track 20.8 -> 7.33 mm, vias 1 -> 0
- net RX_D0: track 6.63 -> 18.4 mm, vias 1 -> 2
- net A0: track 14.6 -> 3.93 mm, vias 1 -> 0
- net D4: track 9.75 -> 19.9 mm
- net D5: track 12.2 -> 20.4 mm
- net SDA: track 16.5 -> 8.53 mm, vias 1 -> 0
- net A6: track 0.00 -> 7.47 mm, vias 0 -> 1
- net MISO: track 21.6 -> 15.9 mm
- net A5: track 3.39 -> 8.75 mm
- net SCL: track 15.5 -> 10.7 mm
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Other:
- board text added: "D51"
- board text added: "build D51 009"
- board text removed: "C13"
- board text removed: "D51 build 008 2018"
- board text removed: "R6"
- board text removed: "build D51 008"
