File: MINI_SAM_D51_013.brd (EAGLE design)
At the start: 25.4 x 40.4 mm, 32 parts, among them IC2 PRTR5V0U2X, IC4 ATSAMD51G_TQFN48, J1 MOLEX_47346-100147346, J2 CORTEX_DEBUG_PTH, SW1 KMS233GLFG, SW2 KMS233GLFG, U1 GD25x16

Commit message: Adding revisions
Parts:
- removed L: (no value), microbuilder:CHIPLED_0603_NOOUTLINE
- added J5: 1X8_HEADER_1.27MMCAST, Shockley_Custom:1X8_HEADER_1.27MM_CASTELLATED
- added LED: (no value), microbuilder:CHIPLED_0805_NOOUTLINE
- J2: value CORTEX_DEBUG_PTH -> 1X5_HEADER_1.27MMCAST; device SparkFun-Connectors:2X5-PTH-1.27MM -> Shockley_Custom:1X5_HEADER_1.27MM_CASTELLATED
- J3: value (none) -> 1X8_HEADER_1.27MMCAST; device pinhead+:1X11_SMT -> Shockley_Custom:1X8_HEADER_1.27MM_CASTELLATED
- J4: value (none) -> 1X5_HEADER_1.27MMCAST; device pinhead+:1X11_SMT -> Shockley_Custom:1X5_HEADER_1.27MM_CASTELLATED
- moved J4 15.1 mm to (22.2, 19.2), flipped to the top, turned to 101.5 degrees
- moved J3 11.6 mm to (5.60, 8.25), flipped to the top, turned to 267.8 degrees
- moved U$3 11.2 mm to (5.70, 25.0)
- moved C11 8.95 mm to (12.0, 17.1), flipped to the bottom, turned to 180 degrees
- moved VREG 8.55 mm to (12.0, 19.9), flipped to the bottom, turned to 180 degrees
- moved R2 7.36 mm to (12.0, 27.7), flipped to the bottom, turned to 180 degrees
- moved R8 7.34 mm to (12.0, 15.5), flipped to the bottom, turned to 180 degrees
- moved C10 6.93 mm to (12.0, 23.8), flipped to the bottom, turned to 180 degrees
- moved C7 3.00 mm to (17.0, 10.6)
- moved R5 3.00 mm to (14.0, 10.6)
- moved J2 1.82 mm to (1.77, 19.2), turned to 258.5 degrees
- moved SW1 0.15 mm to (8.07, 1.65)
- moved SW2 0.15 mm to (15.9, 1.65)
- turned C12 to 270 degrees
- turned R4 to 270 degrees
Connections:
- removed net A6_D2: IC4.12, J3.8
- removed net D10: IC4.29
- removed net D11: IC4.30
- removed net D12: IC4.32
- removed net D13: IC4.31, R2.2
- removed net D9: IC4.28, R5.2, SW2.3, SW2.4
- new net A6: IC4.12, J5.P8
- new net BUTTON_D6: IC4.1, R5.2, SW2.2, SW2.3
- new net D14: IC4.24, R2.2
- net !RESET: now also J2.P4; no longer J2.10, J4.8
- net A0: now also J5.P1; no longer J3.2
- net A1: now also IC4.7, J5.P3; no longer IC4.10, J3.3
- net A2: now also IC4.8, J5.P4; no longer IC4.7, J3.4
- net A3: now also IC4.9, J5.P5; no longer IC4.8, J3.5
- net A4: now also IC4.10, J5.P6; no longer IC4.9, J3.6
- net A5: now also J5.P7; no longer J3.7
- net AREF: now also J5.P2; no longer J3.1
- net D3: now also IC4.28, J3.P3; no longer IC4.37, J4.5
- net D4: now also IC4.29, J3.P4; no longer IC4.23, J4.4
- net D5: now also IC4.30, J3.P5; no longer IC4.24, J4.3
- net GND: now also J2.P5, J4.P1, LED.C; no longer J2.3, J2.5, J3.11, L.C
- net MISO: now also J3.P7; no longer J4.10
- net MOSI: now also IC4.37, J3.P6; no longer IC4.1, J4.9
- net N$3: now also LED.A; no longer L.A
- net RX_D0: now also J3.P1; no longer J4.1
- net SCK: now also J3.P8; no longer J4.11
- net SCL: now also J4.P5; no longer J4.6
- net SDA: now also J4.P4; no longer J4.7
- net SWCLK: now also J2.P2; no longer J2.4
- net SWDIO: now also J2.P1; no longer J2.2
- net TX_D1: now also J3.P2; no longer J4.2
- net VDD: now also J2.P3, J4.P2, SW2.1; no longer J2.1, J3.9, SW2.5
- net VIN: now also J4.P3; no longer J3.10
Routing:
- net VDD: track 86.6 -> 14.3 mm, vias 7 -> 8
- net D9: track 40.6 -> 0.00 mm, vias 4 -> 0
- net VIN: track 9.79 -> 40.8 mm, vias 1 -> 0
- net TX_D1: track 1.79 -> 23.4 mm
- net BUTTON_D6: track 0.00 -> 16.3 mm, vias 0 -> 3
- net RX_D0: track 6.63 -> 22.6 mm
- net D3: track 3.71 -> 19.0 mm
- net D4: track 9.75 -> 19.3 mm
- net A6: track 0.00 -> 8.11 mm, vias 0 -> 1
- net D5: track 12.2 -> 19.7 mm
- net A5: track 3.39 -> 9.06 mm
- net AREF: track 20.8 -> 15.1 mm, vias 1 -> 2
- net MISO: track 21.6 -> 15.9 mm
- net D14: track 0.00 -> 5.14 mm, vias 0 -> 1
- net D13: track 4.75 -> 0.00 mm
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- added copper zone on layer 16, net VDD
- removed copper zone on layer 1, net VIN
Other:
- board text added: "!RST"
- board text added: "A0/ VOUT"
- board text added: "A1"
- board text added: "D3~"
- board text added: "D4~"
- board text added: "D51"
- board text added: "D5~"
- board text added: "MEM"
- board text added: "MISO"
- board text added: "MOSI"
- board text added: "RX~"
- board text added: "SCK~"
- board text added: "SCL~"
- board text added: "SDA~"
- board text added: "SWC"
- board text added: "SWD"
- board text added: "TX~"
- board text added: "https:// minisam.cc"
- board text added: "rev: 001 bld: 012"
- board text removed: "-"
- board text removed: "A0"
- board text removed: "C1"
- board text removed: "C12"
- board text removed: "C13"
- board text removed: "C2"
- board text removed: "C3"
- board text removed: "C6"
- board text removed: "C7"
- board text removed: "C8"
- board text removed: "C9"
- board text removed: "CORTEX DBG"
- board text removed: "D51 build 008 2018"
- board text removed: "FB1"
- board text removed: "IC1"
- board text removed: "JP1"
- board text removed: "R3"
- board text removed: "R4"
- board text removed: "R5"
- board text removed: "R6"
- board text removed: "RGB"
- board text removed: "RST"
- board text removed: "RX"
- board text removed: "TX"
- board text removed: "a"
- board text removed: "build D51 008"
- board text removed: "m.cc"
- board text removed: "minis"
- board text removed: "~A1"
- board text removed: "~D3"
- board text removed: "~D4"
- board text removed: "~D5"
- board text removed: "~MISO"
- board text removed: "~MOSI"
- board text removed: "~SCK"
