File: MINI_SAM_D51_017.brd (EAGLE design)
At the start: 25.4 x 40.4 mm, 32 parts, among them J1 MOLEX_47346-100147346, J2 1X5_HEADER_1.27MMCAST, J3 1X8_HEADER_1.27MMCAST, J4 1X5_HEADER_1.27MMCAST, J5 1X8_HEADER_1.27MMCAST, SW1 KMS233GLFG, SW2 KMS233GLFG, U1 ATSAMD51G_TQFN48, U2 QSPI NOR FLASH 2MiB 2x3mm USO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

Commit message: Updated Board Designs
Added new design revisions
Parts:
- LED: value Easily mounted up-sdie down. -> VLRK31Q1R2-GS08; device microbuilder:CHIPLED_0805_NOOUTLINE -> Shockley_Custom:REVERSE_MOUNT_LED
- R5: value 220Ω -> 120Ω
- moved U$3 9.96 mm to (6.00, 24.1)
- moved R5 3.15 mm to (12.0, 24.5)
- moved R6 1.75 mm to (12.0, 16.5)
- moved C10 1.60 mm to (12.0, 17.9)
- moved VREG 1.40 mm to (12.0, 20.8)
- moved C9 1.35 mm to (12.0, 23.4)
- moved D1 0.36 mm to (11.0, 30.4)
- moved D2 0.36 mm to (13.0, 30.4)
- moved J1 0.25 mm to (12.0, 36.8)
- turned LED to 0 degrees
Routing:
- net D14: track 4.89 -> 1.35 mm
- net SWCLK: track 18.0 -> 16.4 mm
- net VDD: track 21.5 -> 20.0 mm
- net N$3: track 1.32 -> 2.60 mm
- net VHI: track 14.5 -> 15.7 mm
- net GND: track 21.8 -> 20.7 mm, vias 10 -> 9
- net VUSB: track 1.98 -> 2.48 mm
Other:
- outline, holes or cut-outs redrawn
- board text added: "LED"
- board text added: "rev: 017 bld: 001"
- board text removed: "rev: 016 bld: 001"
