File: MINI_SAM_D51_017.sch (EAGLE design)
At the start: 31 parts, among them J1 MOLEX_47346-100147346, J2 1X5_HEADER_1.27MMCAST, J3 1X8_HEADER_1.27MMCAST, J4 1X5_HEADER_1.27MMCAST, J5 1X8_HEADER_1.27MMCAST, SW1 KMS233GLFG, SW2 KMS233GLFG, U1 ATSAMD51G_TQFN48, U2 QSPI NOR FLASH 2MiB 2x3mm USO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

Commit message: Updated Board Designs
Added new design revisions
Parts:
- LED: value Easily mounted up-sdie down. -> VLRK31Q1R2-GS08; device microbuilder:LED0805_NOOUTLINE -> Shockley_Custom:REVERSEMOUNTLED
- R5: value 220Ω -> 120Ω
Other:
- moved on the sheet: LED
