File: MINI_SAM_D51_r002_b002.sch (EAGLE design)
At the start: 31 parts, among them J1 MOLEX_47346-100147346, J2 1X5_HEADER_1.27MMCAST, J3 1X8_HEADER_1.27MMCAST, J4 1X5_HEADER_1.27MMCAST, J5 1X8_HEADER_1.27MMCAST, SW1 KMS233GLFG, SW2 KMS233GLFG, U1 ATSAMD51G_TQFN48, U2 QSPI NOR FLASH 2MiB 2x3mm USO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

Commit message: Updated Board Designs
Added new design revisions
Parts:
- added JP1, JP4: (no value), pinhead+:PINHD-1X51X05_SMT
- added JP2: (no value), pinhead+:PINHD-1X61X06_SMT
- added JP3: (no value), pinhead+:PINHD-1X6REV
- LED: value Easily mounted up-sdie down. -> VLRK31Q1R2-GS08; device microbuilder:LED0805_NOOUTLINE -> Shockley_Custom:REVERSEMOUNTLED
- R5: value 220Ω -> 120Ω
Connections:
- net D14 renamed D6
- removed net A6: J5.P$8, U1G$1.PA07/I7/AIN7/SERCOM0.3
- new net A6_D2: J5.P$8, JP1.3, U1G$1.PA07/I7/AIN7/SERCOM0.3
- net !RESET: now also JP4.3
- net A0: now also JP2.6
- net A1: now also JP2.4
- net A2: now also JP2.3
- net A3: now also JP2.1
- net A4: now also JP1.5
- net A5: now also JP2.2
- net AREF: now also JP2.5
- net BAT: now also J4.P$2, JP1.4; no longer J4.P$3
- net D3: now also JP4.1
- net D4: now also JP3.1
- net D5: now also JP3.3
- net GND: now also JP4.5
- net MISO: now also JP3.5
- net MOSI: now also JP3.4
- net RX_D0: now also JP4.2
- net SCK: now also JP3.6
- net SCL: now also JP1.2
- net SDA: now also JP1.1
- net TX_D1: now also JP3.2
- net VDD: now also J4.P$3, JP4.4; no longer J4.P$2
Other:
- moved on the sheet: LED
